File: inverter comms/inverter comms.kicad_pcb (KiCad board)
At the start: 2 copper layers, 68.5 x 38.5 mm, 33 parts, among them J1 RJ45 - IN, J2 RJ45 - OUT, J3 USB_C_Receptacle_USB2.0_14P, J4 Screw_Terminal_01x02, U1 ESP32-S3-WROOM-1, U2 MAX485E, U3 LM1117DT-3.3

Commit message: V1
Parts:
- U2: footprint Package_SO:SOIC-8-N7_3.9x4.9mm_P1.27mm -> Package_SO:SOIC-8_3.9x4.9mm_P1.27mm
- moved U2 0.30 mm to (153.2, 79.5)
Routing:
- net BUS B: track 17.3 -> 24.7 mm
