File: inverter comms/inverter comms.kicad_sch (KiCad schematic)
At the start: 33 parts, among them J1 RJ45 - IN, J2 RJ45 - OUT, J3 USB_C_Receptacle_USB2.0_14P, J4 Screw_Terminal_01x02, U1 ESP32-S3-WROOM-1, U2 MAX485E, U3 LM1117DT-3.3

Commit message: V1
Parts:
- U2: footprint Package_SO:SOIC-8-N7_3.9x4.9mm_P1.27mm -> Package_SO:SOIC-8_3.9x4.9mm_P1.27mm
Changed lines of the file:
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@@
 			)
 		)
-		(property "Footprint" "Package_SO:SOIC-8-N7_3.9x4.9mm_P1.27mm"
+		(property "Footprint" "Package_SO:SOIC-8_3.9x4.9mm_P1.27mm"
 			(at 116.84 83.82 0)
 			(effects
